Commit message: minor

File: src/stretch/config/urdf/stretch.urdf (robot description, URDF)
Before this commit: robot stretch, 62 links, 61 joints
Joints:
- joint camera_joint: origin xyz=0.025036270286076162 -0.012708115233039453 0.018380101739405765 rpy=-0.001966548079939758 0.014351848596652506 -0.05544266656048365 -> xyz=0.0257482922313648 -0.010591850111920613 0.019379855388464873 rpy=-0.00512855822985284 -0.029627674931582026 -0.02431790587555529
- joint joint_arm_l4: origin xyz=-0.25685100006263134 0.001745354475656944 -0.009321156848349905 rpy=1.5760155686307726 0.017699445406025083 -1.5888018080300244 -> xyz=-0.25490668405769307 -0.008127237970279151 -0.005767330274926086 rpy=1.5911243198548901 -0.017207543060219654 -1.5597906715092422
- joint joint_head_pan: origin xyz=0.13737760722587775 0.07364580135320134 -0.012498809596558429 rpy=0.005121023065690289 0.006431089529577383 1.6226013153376 -> xyz=0.13521129739846033 0.07524851227884313 -0.0039765046776770235 rpy=0.0070286539605192155 0.00647849135595302 1.5612432263323943
- joint joint_head_tilt: origin xyz=0.000351096447700929 0.02684289552312893 -0.0513481404827412 rpy=1.5579758187097514 0.044051992514639426 -0.021397790601784816 -> xyz=0.003182762594451201 0.028122604304064817 -0.061919148952510876 rpy=1.601177353631352 -0.05110972907209299 -0.04867230184589155
- joint joint_mast: origin xyz=-0.06907295519617487 0.13572310789327843 0.02748820981449078 rpy=1.5709474453273709 -0.013818799206169796 0.029932700168379678 -> xyz=-0.0719020049764669 0.13697414498656316 0.036632581953753934 rpy=1.5992656529246831 0.002153566415689756 0.00016049306152166043
